Commit message: Mejoras en Vision, Errores en movimiento

File: src/panda_ws/panda_description/urdf/sensors.xacro (robot description, xacro)
@@ -23,5 +23,5 @@
     </link>
     <joint name="camera_joint" type="fixed">
-        <origin xyz="0.9 0 1.24" rpy="0.0 0.0 0.0"/>
+        <origin xyz="0.60 0 1.12" rpy="0.0 0.0 0.0"/>
         <parent link="panda_link0"/>
         <child link="camera_link"/>

Commit message: Sigue con Errores sobretodo el tema de grasping

File: src/panda_ws/panda_description/urdf/sensors.xacro (robot description, xacro)
@@ -23,5 +23,5 @@
     </link>
     <joint name="camera_joint" type="fixed">
-        <origin xyz="0.60 0 1.12" rpy="0.0 0.0 0.0"/>
+        <origin xyz="0.60 0 1.12" rpy="0.0 1.5708 0.0"/>
         <parent link="panda_link0"/>
         <child link="camera_link"/>
@@ -35,5 +35,5 @@
     <gazebo reference="camera_link">
         <sensor name="camera" type="rgbd_camera">
-            <pose>0 0 0 0 1.57 0</pose>
+            <pose>0 0 0 0 0 0</pose>
             <visualize>true</visualize>
             <update_rate>10.0</update_rate>
